Commit message: updated urdf and odrive readme

File: urdf/robot.urdf (robot description, URDF)
Before this commit: robot onshape, 7 links, 6 joints
Joints:
- joint back_left_wheel: origin xyz=0.346667 -1.31839e-16 0.325 rpy=-3.14159 2.47388e-14 3.14159 -> xyz=0.346667 -1.04083e-16 0.325 rpy=-3.14159 2.47943e-14 3.14159
- joint back_leg: origin xyz=-0.15 0.2 -0.04 rpy=1.5708 2.19171e-16 1.5708 -> xyz=-0.15 0.2 -0.04 rpy=1.5708 -3.33067e-16 1.5708
- joint back_right_wheel: origin xyz=0.346667 -1.04083e-16 -0.025 rpy=3.15653e-15 1.23664e-14 -3.1003 -> xyz=0.346667 -1.04083e-16 -0.025 rpy=3.15882e-15 1.24219e-14 -3.1003
- joint front_left_wheel: origin xyz=0.346667 -9.02056e-17 0.325 rpy=-3.14159 4.83799e-16 -0.0340289 -> xyz=0.346667 -1.80411e-16 0.325 rpy=-3.14159 -1.77836e-16 -2.35619
- joint front_leg: origin xyz=-0.15 -0.2 -0.04 rpy=-1.5708 9.02056e-17 -1.5708 -> xyz=-0.15 -0.2 -0.04 rpy=-1.5708 -1.66533e-16 -1.5708
- joint front_right_wheel: origin xyz=0.346667 -1.11022e-16 -0.025 rpy=1.39509e-16 4.06919e-17 -0.0872665 -> xyz=0.346667 -1.66533e-16 -0.025 rpy=1.41928e-16 1.30419e-17 -0.0872665

Commit message: swapped robot front and back

File: urdf/robot.urdf (robot description, URDF)
Before this commit: robot onshape, 7 links, 6 joints
Joints:
- joint back_left_wheel: child wheel_4 -> wheel_3; origin xyz=0.346667 -1.04083e-16 0.325 rpy=-3.14159 2.47943e-14 3.14159 -> xyz=0.346667 -1.11022e-16 -0.025 rpy=2.10385e-17 -2.31218e-16 3.05433
- joint back_leg: origin xyz=-0.15 0.2 -0.04 rpy=1.5708 -3.33067e-16 1.5708 -> xyz=0.15 0.2 -0.04 rpy=-1.5708 2.52435e-28 1.5708
- joint back_right_wheel: child wheel_3 -> wheel_4; origin xyz=0.346667 -1.04083e-16 -0.025 rpy=3.15882e-15 1.24219e-14 -3.1003 -> xyz=0.346667 -1.11022e-16 0.325 rpy=-3.14159 -1.13436e-16 0.785398
- joint front_left_wheel: child wheel_2 -> wheel; origin xyz=0.346667 -1.80411e-16 0.325 rpy=-3.14159 -1.77836e-16 -2.35619 -> xyz=0.346667 -1.11022e-16 -0.025 rpy=3.012e-15 1.23012e-14 0.0412877
- joint front_leg: origin xyz=-0.15 -0.2 -0.04 rpy=-1.5708 -1.66533e-16 -1.5708 -> xyz=0.15 -0.2 -0.04 rpy=1.5708 -8.28304e-30 -1.5708
- joint front_right_wheel: child wheel -> wheel_2; origin xyz=0.346667 -1.66533e-16 -0.025 rpy=1.41928e-16 1.30419e-17 -0.0872665 -> xyz=0.346667 -1.11022e-16 0.325 rpy=-3.14159 2.46677e-14 -2.63678e-15
